File: PCB/Capstone.kicad_pcb (KiCad board)
At the start: 2 copper layers, 0 parts

Commit message: Annotate schematic, simplify transmit circuit, shuffle receive opamp stages, reorder buttons so they match net names, reorder connectors to simplify routing, begin arranging parts on PCB
Parts:
- added C1: 10uF, Capacitors_SMD:C_0805_HandSoldering, F.Cu at (45.7, 34.8)
- added C10: 10uF, Capacitors_SMD:C_0805_HandSoldering, F.Cu at (117.3, 48.3)
- added C100: 10uF, Capacitors_SMD:C_0805_HandSoldering, F.Cu at (213.4, 140.0)
- added C101: 100nF, Capacitors_SMD:C_0603_HandSoldering, F.Cu at (210.1, 147.6)
- added C102: 4.7uF, Capacitors_SMD:C_0603_HandSoldering, F.Cu at (218.0, 141.5)
- added C103: 2.2nF, Capacitors_SMD:C_0603_HandSoldering, F.Cu at (214.4, 150.4)
- added C11: 10uF, Capacitors_SMD:C_0805_HandSoldering, F.Cu at (112.0, 47.2)
- added C12: 10uF, Capacitors_SMD:C_0805_HandSoldering, F.Cu at (88.6, 22.9)
- added C13: 10uF, Capacitors_SMD:C_0805_HandSoldering, F.Cu at (103.6, 22.9)
- added C14: 10uF, Capacitors_SMD:C_0805_HandSoldering, F.Cu at (122.2, 23.4)
- added C15: 330uF, Capacitors_THT:CP_Radial_D6.3mm_P2.50mm, F.Cu at (116.6, 22.1)
- added C16: 330uF, Capacitors_THT:CP_Radial_D6.3mm_P2.50mm, F.Cu at (108.7, 22.1)
- added C17: 1uF, Capacitors_SMD:C_0603_HandSoldering, F.Cu at (113.0, 50.5)
- added C18: 10uF, Capacitors_SMD:C_0805_HandSoldering, F.Cu at (127.3, 50.3)
- added C19: 10uF, Capacitors_SMD:C_0805_HandSoldering, F.Cu at (131.8, 49.0)
- added C2: 10uF, Capacitors_SMD:C_0805_HandSoldering, F.Cu at (54.4, 34.8)
- added C20: 100nF, Capacitors_SMD:C_0603_HandSoldering, F.Cu at (69.6, 130.0)
- added C21: 10uF, Capacitors_SMD:C_0805_HandSoldering, F.Cu at (73.2, 130.0)
- added C22: 10uF, Capacitors_SMD:C_0805_HandSoldering, F.Cu at (23.1, 81.5)
- added C23: 10nF, Capacitors_SMD:C_0603_HandSoldering, F.Cu at (50.5, 51.3)
- added C24: 100nF, Capacitors_SMD:C_0603_HandSoldering, F.Cu at (46.5, 84.3)
- added C25: 100nF, Capacitors_SMD:C_0603_HandSoldering, F.Cu at (20.8, 118.9)
- added C26: 100nF, Capacitors_SMD:C_0603_HandSoldering, F.Cu at (21.1, 129.4)
- added C27: 100nF, Capacitors_SMD:C_0603_HandSoldering, F.Cu at (65.5, 108.2)
- added C28: 10uF, Capacitors_SMD:C_0805_HandSoldering, F.Cu at (65.3, 111.5)
- added C29: 10uF, Capacitors_SMD:C_0805_HandSoldering, F.Cu at (156.5, 22.9)
- added C3: 10uF, Capacitors_SMD:C_0805_HandSoldering, F.Cu at (62.7, 35.1)
- added C30: 10uF, Capacitors_SMD:C_1206_HandSoldering, F.Cu at (171.2, 17.0)
- added C31: 10uF, Capacitors_SMD:C_1206_HandSoldering, F.Cu at (174.8, 22.1)
- added C32: 2.2nF, Capacitors_SMD:C_0603_HandSoldering, F.Cu at (167.4, 28.4)
- added C33: 1uF, Capacitors_SMD:C_0805_HandSoldering, F.Cu at (198.9, 48.3)
- added C34: 1uF, Capacitors_SMD:C_0805_HandSoldering, F.Cu at (205.2, 55.4)
- added C35: 10uF, Capacitors_SMD:C_1206_HandSoldering, F.Cu at (199.6, 57.7)
- added C36: 10uF, Capacitors_SMD:C_1206_HandSoldering, F.Cu at (249.9, 19.6)
- added C37: 100nF, Capacitors_SMD:C_0603_HandSoldering, F.Cu at (239.0, 33.3)
- added C38: 220uF, Capacitors_THT:CP_Radial_D10.0mm_P5.00mm, F.Cu at (258.8, 36.3)
- added C39: 220uF, Capacitors_THT:CP_Radial_D10.0mm_P5.00mm, F.Cu at (269.5, 28.7)
- added C4: 330uF, Capacitors_THT:CP_Radial_D6.3mm_P2.50mm, F.Cu at (58.9, 33.5)
- added C40: 220pF, Capacitors_SMD:C_0603_HandSoldering, F.Cu at (243.4, 28.4)
- added C41: 220pF, Capacitors_SMD:C_0603_HandSoldering, F.Cu at (244.3, 37.8)
- added C42: 220pF, Capacitors_SMD:C_0603_HandSoldering, F.Cu at (155.2, 26.9)
- added C43: 10pF, Capacitors_SMD:C_0603_HandSoldering, F.Cu at (246.1, 33.5)
- added C44: 100nF, Capacitors_SMD:C_0603_HandSoldering, F.Cu at (128.5, 70.4)
- added C45: 100nF, Capacitors_SMD:C_0603_HandSoldering, F.Cu at (129.3, 83.2)
- added C46: 100nF, Capacitors_SMD:C_0603_HandSoldering, F.Cu at (109.5, 110.2)
- added C47: 100nF, Capacitors_SMD:C_0603_HandSoldering, F.Cu at (132.3, 83.6)
- added C48: 100nF, Capacitors_SMD:C_0603_HandSoldering, F.Cu at (106.7, 109.8)
- added C49: 2.2nF, Capacitors_SMD:C_0603_HandSoldering, F.Cu at (124.0, 83.0)
- added C5: 100nF, Capacitors_SMD:C_0603_HandSoldering, F.Cu at (47.6, 38.9)
- added C50: 2.2nF, Capacitors_SMD:C_0603_HandSoldering, F.Cu at (114.8, 83.0)
- added C51: 2.2nF, Capacitors_SMD:C_0603_HandSoldering, F.Cu at (104.6, 90.2)
- added C52: 2.2nF, Capacitors_SMD:C_0603_HandSoldering, F.Cu at (104.6, 101.9)
- added C53: 2.2nF, Capacitors_SMD:C_0603_HandSoldering, F.Cu at (114.6, 110.6)
- added C54: 2.2nF, Capacitors_SMD:C_0603_HandSoldering, F.Cu at (123.4, 110.7)
- added C55: 2.2nF, Capacitors_SMD:C_0603_HandSoldering, F.Cu at (132.6, 103.1)
- added C56: 2.2nF, Capacitors_SMD:C_0603_HandSoldering, F.Cu at (133.1, 91.2)
- added C57: 22nF, Capacitors_SMD:C_0603_HandSoldering, F.Cu at (126.5, 83.0)
- added C58: 22nF, Capacitors_SMD:C_0603_HandSoldering, F.Cu at (117.3, 83.0)
- added C59: 22nF, Capacitors_SMD:C_0603_HandSoldering, F.Cu at (104.6, 87.4)
- added C6: 1uF, Capacitors_SMD:C_0603_HandSoldering, F.Cu at (82.3, 44.7)
- added C60: 22nF, Capacitors_SMD:C_0603_HandSoldering, F.Cu at (104.6, 99.3)
- added C61: 22nF, Capacitors_SMD:C_0603_HandSoldering, F.Cu at (112.0, 110.6)
- added C62: 22nF, Capacitors_SMD:C_0603_HandSoldering, F.Cu at (120.9, 110.6)
- added C63: 22nF, Capacitors_SMD:C_0603_HandSoldering, F.Cu at (132.7, 100.3)
- added C64: 22nF, Capacitors_SMD:C_0603_HandSoldering, F.Cu at (133.3, 88.4)
- added C65: 100nF, Capacitors_SMD:C_0603_HandSoldering, F.Cu at (158.8, 107.4)
- added C66: 100nF, Capacitors_SMD:C_0603_HandSoldering, F.Cu at (156.0, 90.4)
- added C67: 100nF, Capacitors_SMD:C_0603_HandSoldering, F.Cu at (151.1, 95.2)
- added C68: 1uF, Capacitors_SMD:C_0603_HandSoldering, F.Cu at (155.1, 93.2)
- added C69: 10uF, Capacitors_SMD:C_0805_HandSoldering, F.Cu at (153.7, 84.6)
- added C7: 1uF, Capacitors_SMD:C_0603_HandSoldering, F.Cu at (90.4, 44.5)
- added C70: 10uF, Capacitors_SMD:C_0805_HandSoldering, F.Cu at (150.1, 89.9)
- added C71: 22nF, Capacitors_SMD:C_0603_HandSoldering, F.Cu at (159.8, 95.1)
- added C72: 22nF, Capacitors_SMD:C_0603_HandSoldering, F.Cu at (153.4, 106.5)
- added C73: 22nF, Capacitors_SMD:C_0603_HandSoldering, F.Cu at (154.8, 97.9)
- added C74: 22nF, Capacitors_SMD:C_0603_HandSoldering, F.Cu at (151.1, 104.1)
- added C75: 22nF, Capacitors_SMD:C_0603_HandSoldering, F.Cu at (159.5, 97.9)
- added C76: 22nF, Capacitors_SMD:C_0603_HandSoldering, F.Cu at (158.4, 103.6)
- added C77: 100nF, Capacitors_SMD:C_0603_HandSoldering, F.Cu at (159.5, 100.2)
- added C78: 100nF, Capacitors_SMD:C_0603_HandSoldering, F.Cu at (153.9, 108.9)
- added C79: 1uF, Capacitors_SMD:C_0603_HandSoldering, F.Cu at (154.8, 100.2)
- added C8: 10uF, Capacitors_SMD:C_0805_HandSoldering, F.Cu at (93.2, 44.7)
- added C80: 10uF, Capacitors_SMD:C_0805_HandSoldering, F.Cu at (149.6, 100.1)
- added C81: 220nF, Capacitors_SMD:C_1206_HandSoldering, F.Cu at (230.6, 89.4)
- added C82: 100nF, Capacitors_SMD:C_0603_HandSoldering, F.Cu at (201.7, 83.8)
- added C83: 10uF, Capacitors_SMD:C_0805_HandSoldering, F.Cu at (205.0, 83.8)
- added C84: 100nF, Capacitors_SMD:C_0603_HandSoldering, F.Cu at (204.2, 94.5)
- added C85: 100nF, Capacitors_SMD:C_1206_HandSoldering, F.Cu at (212.9, 91.4)
- added C86: 100nF, Capacitors_SMD:C_1206_HandSoldering, F.Cu at (256.8, 105.7)
- added C87: 220nF, Capacitors_SMD:C_1206_HandSoldering, F.Cu at (215.4, 80.5)
- added C88: 2.2uF, Capacitors_SMD:C_1210_HandSoldering, F.Cu at (224.0, 86.9)
- added C89: 2.2nF, Capacitors_SMD:C_0603_HandSoldering, F.Cu at (210.6, 84.3)
- added C9: 1uF, Capacitors_SMD:C_0603_HandSoldering, F.Cu at (114.6, 43.7)
- added C90: 100nF, Capacitors_SMD:C_0603_HandSoldering, F.Cu at (200.7, 134.6)
- added C91: 100nF, Capacitors_SMD:C_0603_HandSoldering, F.Cu at (204.7, 124.0)
- added C92: 100nF, Capacitors_SMD:C_0603_HandSoldering, F.Cu at (206.2, 141.7)
- added C93: 10uF, Capacitors_SMD:C_0805_HandSoldering, F.Cu at (209.3, 141.7)
- added C94: 100nF, Capacitors_SMD:C_1206_HandSoldering, F.Cu at (256.8, 111.0)
- added C95: 150nF, Capacitors_SMD:C_0603_HandSoldering, F.Cu at (220.0, 136.7)
- added C96: 150nF, Capacitors_SMD:C_0603_HandSoldering, F.Cu at (220.5, 128.8)
- added C97: 150nF, Capacitors_SMD:C_0603_HandSoldering, F.Cu at (214.6, 118.6)
- added C98: 150nF, Capacitors_SMD:C_0603_HandSoldering, F.Cu at (206.2, 127.0)
- added C99: 100nF, Capacitors_SMD:C_0603_HandSoldering, F.Cu at (213.1, 136.7)
- added D1: LED_ABGR, Parts:CLMVC-FKA, F.Cu at (27.7, 81.3)
- added D2: 560mV 2.1A, Diodes_SMD:D_SOD-123F, F.Cu at (178.6, 25.9)
- added D3: 560mV 2.1A, Diodes_SMD:D_SOD-123F, F.Cu at (243.8, 24.4)
- added D4: 600mV 200mA, Diodes_SMD:D_SOD-523, F.Cu at (252.0, 104.9)
- added D5: 600mV 200mA, Diodes_SMD:D_SOD-523, F.Cu at (252.0, 106.4)
- added D6: 2.7V, Diodes_SMD:D_SOD-123, F.Cu at (229.1, 87.1)
- added D7: 600mV 200mA, Diodes_SMD:D_SOD-523, F.Cu at (255.0, 115.8)
- added D8: 600mV 200mA, Diodes_SMD:D_SOD-523, F.Cu at (255.0, 114.3)
- added H1: MountingHole_Pad, Mounting_Holes:MountingHole_4mm_Pad_Via, F.Cu at (33.5, 20.8)
- added H2: MountingHole_Pad, Mounting_Holes:MountingHole_4mm_Pad_Via, F.Cu at (42.7, 161.0)
- added J1: S2B-PH-SM4-TB, Parts:JST_S2B-PH-SM4-TB, F.Cu at (26.9, 31.2)
- added J10: DNP, Pin_Headers:Pin_Header_Straight_1x03_Pitch2.54mm, F.Cu at (198.9, 122.7)
- added J11: DNP, Pin_Headers:Pin_Header_Straight_1x03_Pitch2.54mm, F.Cu at (194.6, 124.0)
- added J12: PH1-08-UA, Pin_Headers:Pin_Header_Straight_1x08_Pitch2.54mm, F.Cu at (82.3, 100.6)
- added J13: DNP, Pin_Headers:Pin_Header_Straight_1x08_Pitch2.54mm, F.Cu at (81.8, 77.7)
- added J14: DNP, Pin_Headers:Pin_Header_Straight_1x02_Pitch2.54mm, F.Cu at (272.5, 37.6)
- added J15: DNP, Pin_Headers:Pin_Header_Straight_1x03_Pitch2.54mm, F.Cu at (188.7, 85.3)
- added J2: TRANSDUCER, Pin_Headers:Pin_Header_Straight_1x02_Pitch2.54mm, F.Cu at (267.7, 108.2)
- added J3: DNP, Pin_Headers:Pin_Header_Straight_1x02_Pitch2.54mm, F.Cu at (127.3, 24.6)
- added J4: PH1-08-UA, Pin_Headers:Pin_Header_Straight_1x08_Pitch2.54mm, F.Cu at (17.8, 60.2)
- added J5: DNP, Pin_Headers:Pin_Header_Straight_1x08_Pitch2.54mm, F.Cu at (100.3, 140.2)
- added J6: DNP, Pin_Headers:Pin_Header_Straight_1x02_Pitch2.54mm, F.Cu at (37.3, 121.7)
- added J7: DNP, Pin_Headers:Pin_Header_Straight_1x02_Pitch2.54mm, F.Cu at (194.1, 52.1)
- added J8: DNP, Pin_Headers:Pin_Header_Straight_1x03_Pitch2.54mm, F.Cu at (194.3, 138.4)
- added J9: DNP, Pin_Headers:Pin_Header_Straight_1x02_Pitch2.54mm, F.Cu at (183.6, 21.6)
- added JP1: 0, Parts:SolderJumper_0603, F.Cu at (42.9, 33.5)
- added JP2: 0, Parts:SolderJumper_0603, F.Cu at (51.8, 33.5)
- added JP3: 0, Parts:SolderJumper_0603, F.Cu at (83.6, 21.3)
- added JP4: 0, Parts:SolderJumper_0603, F.Cu at (101.1, 21.8)
- added JP5: 0, Parts:SolderJumper_0603, F.Cu at (156.2, 19.1)
- added JP6: 0, Parts:SolderJumper_0603, F.Cu at (179.1, 17.5)
- added JP7: 0, Parts:SolderJumper_0603, F.Cu at (243.9, 19.3)
- added JP8: 0, Parts:SolderJumper_0603, F.Cu at (252.0, 33.0)
- added L1: 2.2uH, Inductors:Inductor_Taiyo-Yuden_MD-3030, F.Cu at (48.5, 31.2)
- added L2: 100nH, Resistors_SMD:R_0805_HandSoldering, F.Cu at (123.3, 48.0)
- added L3: 2.2uH, Inductors:Inductor_Taiyo-Yuden_MD-3030, F.Cu at (97.5, 22.9)
- added L4: 100nH, Resistors_SMD:R_0805_HandSoldering, F.Cu at (123.7, 43.7)
- added L5: 10uH, Parts:NRS6045T100MMGK, F.Cu at (163.1, 19.1)
- added L6: 150uH, Parts:SRU1048-151Y, F.Cu at (261.9, 21.3)
- added NT1: Net-Tie_2, Parts:NetTie-2, F.Cu at (50.3, 38.6)
- added NT2: Net-Tie_2, Parts:NetTie-2, F.Cu at (91.9, 26.9)
- added NT3: Net-Tie_2, Parts:NetTie-2, F.Cu at (162.6, 30.5)
- added NT4: Net-Tie_2, Parts:NetTie-2, F.Cu at (247.7, 31.0)
- added NT5: Net-Tie_2, Parts:NetTie-2, F.Cu at (119.9, 79.2)
- added Q1: SSM6K361NU, Parts:UDFN6-FET-PAD, F.Cu at (249.9, 36.3)
- added R1: 100m, Resistors_SMD:R_0805_HandSoldering, F.Cu at (118.3, 45.7)
- added R10: 47, Resistors_SMD:R_0603_HandSoldering, F.Cu at (28.7, 91.2)
- added R11: 30, Resistors_SMD:R_0603_HandSoldering, F.Cu at (28.7, 86.6)
- added R12: 1k, Resistors_SMD:R_0603_HandSoldering, F.Cu at (43.4, 65.0)
- added R13: 1k, Resistors_SMD:R_0603_HandSoldering, F.Cu at (15.7, 65.8)
- added R14: 470k, Resistors_SMD:R_0603_HandSoldering, F.Cu at (52.3, 81.5)
- added R15: 1k, Resistors_SMD:R_0603_HandSoldering, F.Cu at (30.7, 64.5)
- added R16: 470k, Resistors_SMD:R_0603_HandSoldering, F.Cu at (52.8, 84.8)
- added R17: 220k, Resistors_SMD:R_0603_HandSoldering, F.Cu at (46.0, 93.5)
- added R18: 3.3k, Resistors_SMD:R_0603_HandSoldering, F.Cu at (53.6, 88.9)
- added R19: 27k, Resistors_SMD:R_0603_HandSoldering, F.Cu at (53.6, 92.5)
- added R2: 100m, Resistors_SMD:R_0805_HandSoldering, F.Cu at (127.8, 47.0)
- added R20: 10k, Resistors_SMD:R_0603_HandSoldering, F.Cu at (66.8, 96.0)
- added R21: 86.6k, Capacitors_SMD:C_0603_HandSoldering, F.Cu at (173.0, 24.9)
- added R22: 10k, Capacitors_SMD:C_0603_HandSoldering, F.Cu at (156.5, 30.0)
- added R23: 10k, Capacitors_SMD:C_0603_HandSoldering, F.Cu at (168.7, 25.4)
- added R24: 220k, Capacitors_SMD:C_0603_HandSoldering, F.Cu at (194.3, 48.8)
- added R25: 30k, Capacitors_SMD:C_0603_HandSoldering, F.Cu at (203.5, 51.8)
- added R26: 392k, Capacitors_SMD:C_0603_HandSoldering, F.Cu at (248.2, 22.9)
- added R27: 10k, Capacitors_SMD:C_0603_HandSoldering, F.Cu at (249.1, 41.4)
- added R28: 100, Capacitors_SMD:C_0603_HandSoldering, F.Cu at (247.4, 16.8)
- added R29: 220k, Capacitors_SMD:C_0603_HandSoldering, F.Cu at (252.2, 23.6)
- added R3: 20k, Resistors_SMD:R_0603_HandSoldering, F.Cu at (45.2, 51.3)
- added R30: 100m, Capacitors_SMD:C_0603_HandSoldering, F.Cu at (243.6, 41.7)
- added R31: 20k, Capacitors_SMD:C_0603_HandSoldering, F.Cu at (254.3, 41.1)
- added R32: 10k, Resistors_SMD:R_0603_HandSoldering, F.Cu at (95.6, 80.5)
- added R33: 10k, Resistors_SMD:R_0603_HandSoldering, F.Cu at (95.1, 83.6)
- added R34: 10k, Resistors_SMD:R_0603_HandSoldering, F.Cu at (95.8, 89.9)
- added R35: 10k, Resistors_SMD:R_0603_HandSoldering, F.Cu at (95.6, 86.6)
- added R36: 10k, Resistors_SMD:R_0603_HandSoldering, F.Cu at (95.4, 93.2)
- added R37: 10k, Resistors_SMD:R_0603_HandSoldering, F.Cu at (95.3, 102.1)
- added R38: 1k, Resistors_SMD:R_0603_HandSoldering, F.Cu at (95.8, 96.0)
- added R39: 10k, Resistors_SMD:R_0603_HandSoldering, F.Cu at (95.5, 99.1)
- added R4: 3.3k, Resistors_SMD:R_0603_HandSoldering, F.Cu at (42.2, 124.5)
- added R40: 10k, Resistors_SMD:R_0603_HandSoldering, F.Cu at (95.6, 105.2)
- added R41: 10k, Resistors_SMD:R_0603_HandSoldering, F.Cu at (137.6, 97.0)
- added R42: 10k, Resistors_SMD:R_0603_HandSoldering, F.Cu at (137.6, 94.2)
- added R43: 10k, Resistors_SMD:R_0603_HandSoldering, F.Cu at (137.6, 92.5)
- added R44: 15k, Resistors_SMD:R_0603_HandSoldering, F.Cu at (221.7, 94.3)
- added R45: 75k, Resistors_SMD:R_0603_HandSoldering, F.Cu at (230.9, 98.8)
- added R46: 15k, Resistors_SMD:R_0603_HandSoldering, F.Cu at (220.6, 91.4)
- added R47: 15k, Resistors_SMD:R_0603_HandSoldering, F.Cu at (200.9, 88.6)
- added R48: 1k, Resistors_SMD:R_0603_HandSoldering, F.Cu at (217.2, 93.4)
- added R49: 10k, Resistors_SMD:R_0603_HandSoldering, F.Cu at (199.6, 91.8)
- added R5: 30, Resistors_SMD:R_0603_HandSoldering, F.Cu at (26.9, 88.1)
- added R50: 220k, Resistors_SMD:R_0603_HandSoldering, F.Cu at (211.1, 78.5)
- added R51: 10, Resistors_SMD:R_0603_HandSoldering, F.Cu at (220.5, 83.8)
- added R52: 220k, Resistors_SMD:R_0603_HandSoldering, F.Cu at (209.0, 84.2)
- added R53: 47k, Resistors_SMD:R_0603_HandSoldering, F.Cu at (218.4, 131.8)
- added R54: 47k, Resistors_SMD:R_0603_HandSoldering, F.Cu at (216.6, 121.4)
- added R55: 7.5k, Resistors_SMD:R_0603_HandSoldering, F.Cu at (210.3, 124.0)
- added R56: 7.5k, Resistors_SMD:R_0603_HandSoldering, F.Cu at (208.0, 133.9)
- added R57: 2.7k, Resistors_SMD:R_0603_HandSoldering, F.Cu at (217.9, 134.9)
- added R58: 2.7k, Resistors_SMD:R_0603_HandSoldering, F.Cu at (216.7, 123.4)
- added R59: 330, Resistors_SMD:R_0603_HandSoldering, F.Cu at (210.6, 119.1)
- added R6: 3.3k, Resistors_SMD:R_0603_HandSoldering, F.Cu at (42.1, 121.7)
- added R60: 330, Resistors_SMD:R_0603_HandSoldering, F.Cu at (203.5, 128.4)
- added R61: 1k, Resistors_SMD:R_0603_HandSoldering, F.Cu at (216.9, 138.3)
- added R62: 1k, Resistors_SMD:R_0603_HandSoldering, F.Cu at (218.4, 126.7)
- added R63: 1k, Resistors_SMD:R_0603_HandSoldering, F.Cu at (212.9, 122.2)
- added R64: 1k, Resistors_SMD:R_0603_HandSoldering, F.Cu at (209.9, 127.3)
- added R65: 30k, Resistors_SMD:R_0603_HandSoldering, F.Cu at (214.4, 157.0)
- added R66: 10, Resistors_SMD:R_0603_HandSoldering, F.Cu at (217.2, 144.5)
- added R67: 30k, Resistors_SMD:R_0603_HandSoldering, F.Cu at (214.4, 152.9)
- added R68: 10k, Resistors_SMD:R_1206_HandSoldering, F.Cu at (262.9, 109.4)
- added R7: 10k, Resistors_SMD:R_0603_HandSoldering, F.Cu at (35.6, 64.5)
- added R8: 47, Resistors_SMD:R_0603_HandSoldering, F.Cu at (25.1, 90.9)
- added R9: 30k, Resistors_SMD:R_0603_HandSoldering, F.Cu at (50.5, 53.3)
- added SW1: SW_Push, Parts:PTS645SK43SM, F.Cu at (46.5, 71.4)
- added SW2: SW_Push, Parts:PTS645SK43SM, F.Cu at (21.8, 71.6)
- added SW3: SW_Push, Parts:PTS645SK43SM, F.Cu at (34.0, 71.4)
- added U1: TPS63031, Parts:WSON10-PAD, F.Cu at (48.5, 34.8)
- added U10: AP2204K-ADJ, Parts:SOT23-5, F.Cu at (198.9, 52.8)
- added U11: LM3478, Parts:SSOP8, F.Cu at (252.7, 28.2)
- added U12: 10CL010, Parts:EQFP144-PAD, F.Cu at (118.7, 96.8)
- added U13: ECS-5032MV, Parts:ECS-5032MV, F.Cu at (128.5, 73.7)
- added U14: TSX9291, Parts:SOT23-5, F.Cu at (202.9, 91.7)
- added U15: LTC6090-5, Parts:SOIC8-PAD, F.Cu at (227.6, 93.7)
- added U16: AD5450, Parts:TSOT8, F.Cu at (197.6, 85.3)
- added U17: ADA4522-1, Parts:SSOP8, F.Cu at (214.9, 83.3)
- added U18: MAX5394L, Parts:TDFN8-PAD, F.Cu at (202.9, 132.1)
- added U19: MAX5394L, Parts:TDFN8-PAD, F.Cu at (208.0, 121.7)
- added U2: TCR2EF25, Parts:SOT23-5, F.Cu at (87.4, 44.5)
- added U20: MAX11116, Parts:SOT23, F.Cu at (202.2, 141.0)
- added U21: TLV3544, Parts:SSOP14, F.Cu at (214.6, 128.5)
- added U22: MCP6L1, Parts:SOT23-5, F.Cu at (213.6, 147.3)
- added U3: TPS62262, Parts:WSON6-2x2-PAD, F.Cu at (92.5, 22.6)
- added U4: BMD-360, Parts:BMD-360, F.Cu at (62.2, 129.3)
- added U5: MIC841N, Parts:SOT353, F.Cu at (46.5, 88.9)
- added U6: ENS210, Parts:QFN4-PAD, F.Cu at (25.1, 118.9)
- added U7: W25Q80DV, Parts:SOIC8, F.Cu at (69.6, 101.1)
- added U8: LIS2DE12, Parts:LGA12, F.Cu at (25.4, 129.3)
- added U9: LMR62421, Parts:WSON6-3x3-PAD, F.Cu at (162.3, 25.9)
Routing:
- net GND: track 0.00 -> 84.2 mm
- net +3V3-LN: track 0.00 -> 53.3 mm
- net +50V: track 0.00 -> 34.0 mm
- net /Receive/MIDRAIL: track 0.00 -> 24.6 mm
- net /Transmit/MIDRAIL: track 0.00 -> 21.4 mm
- net +3V3: track 0.00 -> 18.0 mm
- net Net-(C85-Pad2): track 0.00 -> 10.6 mm
- net TRANSMIT-ENABLE: track 0.00 -> 10.4 mm
- net Net-(C89-Pad1): track 0.00 -> 10.2 mm
- net Net-(R44-Pad2): track 0.00 -> 9.95 mm
- net Net-(C103-Pad1): track 0.00 -> 8.84 mm
- net Net-(U14-Pad3): track 0.00 -> 7.04 mm
- net Net-(R51-Pad1): track 0.00 -> 7.03 mm
- net Net-(R66-Pad2): track 0.00 -> 6.22 mm
- net Net-(D4-Pad1): track 0.00 -> 5.79 mm
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